File: circuits/stepperboard1.brd (EAGLE design)
At the start: 63.5 x 76.8 mm, 32 parts, among them Q1 FDS5680, Q2 FDS5680, Q3 FDS5680, Q4 FDS5680, Q5 FDS5680, Q6 FDS5680, Q7 FDS5680, Q8 FDS5680

Commit message: h bridge circuit board
Parts:
- added D1, D2, D3, D4, D5, D6, D7, D8: (no value), SparkFun-DiscreteSemi:DIODE-1N4001-KIT
- added LED5: (no value), SparkFun-LED:LED3MM
- added R9: 3.3k, SparkFun-Passives:0603-RES
- added U$5: CW182-ND, spietz-library:CW182-ND
- moved R7 12.7 mm to (70.5, 61.6)
- moved R5 12.1 mm to (67.9, 19.7)
- moved JP2 12.1 mm to (72.0, 37.1)
- moved LED1 12.1 mm to (63.5, 61.6)
- moved LED2 12.1 mm to (63.5, 44.5)
- moved LED3 12.1 mm to (63.5, 5.08)
- moved LED4 12.1 mm to (63.5, 26.0)
- moved R6 12.1 mm to (59.7, 20.3)
- moved R8 12.1 mm to (63.5, 52.1)
Connections:
- removed net N$11: JP2.4, LED3.A, Q7.1, Q7.2, Q7.3, Q8.5, Q8.6, Q8.7, Q8.8, R6.1
- removed net N$12: JP2.3, LED4.A, Q5.1, Q5.2, Q5.3, Q6.5, Q6.6, Q6.7, Q6.8, R5.2
- removed net N$4: JP2.2, LED2.A, Q3.1, Q3.2, Q3.3, Q4.5, Q4.6, Q4.7, Q4.8, R7.1
- removed net N$5: JP2.1, LED1.A, Q1.5, Q1.6, Q1.7, Q1.8, Q2.1, Q2.2, Q2.3, R8.2
- new net A+: D7.A, D8.C, JP2.1, LED1.A, Q1.5, Q1.6, Q1.7, Q1.8, Q2.1, Q2.2, Q2.3, R8.2
- new net A-: D5.C, D6.A, JP2.2, LED2.A, Q3.1, Q3.2, Q3.3, Q4.5, Q4.6, Q4.7, Q4.8, R7.1
- new net B+: D3.C, D4.A, JP2.3, LED4.A, Q5.1, Q5.2, Q5.3, Q6.5, Q6.6, Q6.7, Q6.8, R5.2
- new net B-: D1.A, D2.C, JP2.4, LED3.A, Q7.1, Q7.2, Q7.3, Q8.5, Q8.6, Q8.7, Q8.8, R6.1
- new net N$15: JP8.1, U$5.P$1
- new net N$16: LED5.K, R9.2
- net 12V: now also D1.C, D4.C, D6.C, D7.C, LED5.A, U$5.P$2; no longer JP8.1
- net GND: now also D2.A, D3.A, D5.A, D8.A, R9.1
Routing:
- net B-: track 0.00 -> 113.3 mm
- net A-: track 0.00 -> 106.1 mm, vias 0 -> 2
- net A+: track 0.00 -> 97.0 mm
- net N$11: track 85.5 -> 0.00 mm
- net N$4: track 76.8 -> 0.00 mm, vias 2 -> 0
- net B+: track 0.00 -> 72.2 mm
- net N$5: track 60.6 -> 0.00 mm
- net N$12: track 52.3 -> 0.00 mm
- net 12V: track 91.0 -> 125.0 mm
- net N$15: track 0.00 -> 10.9 mm
- net N$16: track 0.00 -> 5.50 mm
- net N$9: track 17.6 -> 14.2 mm
- net N$1: track 6.77 -> 7.41 mm
- net GND: vias 1 -> 3
Other:
- board size 63.5 x 76.8 mm -> 76.2 x 76.8 mm
- board text added: "1"
- board text added: "2"
- board text added: "3"
- board text added: "4"
- board text added: "A+"
- board text added: "A-"
- board text added: "B+"
- board text added: "B-"
- board text added: "BUTTON"
- board text added: "IRF7862"
- board text added: "NO PATENTS NO COPYRIGHTS NO MONEY NO MINING NO PROPERTY"
- board text added: "ON"
- board text added: "ON/OFF"
- board text added: "STEPPER MOTOR CONTROL"
- board text added: "V+"
