File: circuits/dualHbridge.brd (EAGLE design)
At the start: 76.2 x 76.8 mm, 43 parts, among them Q1 FDS5680, Q2 FDS5680, Q3 FDS5680, Q4 FDS5680, Q5 FDS5680, Q6 FDS5680, Q7 FDS5680, Q8 FDS5680

Commit message: h bridge circuit board
Parts:
- removed JP10, JP11, JP12, JP5, JP6, JP9: M01PTH, SparkFun-Connectors:1X01
- removed LED1, LED2, LED3, LED4, LED5: (no value), SparkFun-LED:LED3MM
- removed R5, R6, R7, R8, R9: 3.3k, SparkFun-Passives:0603-RES
- JP1: value (none) -> M01PTH; device SparkFun-Connectors:1X06_NO_SILK -> SparkFun-Connectors:1X01
- JP3: value M01PTH -> (none); device SparkFun-Connectors:1X01 -> SparkFun-Connectors:1X05
- moved JP1 57.3 mm to (15.2, 81.3), turned to 0 degrees
- moved JP3 35.0 mm to (2.54, 36.8), turned to 90 degrees
- moved D7 28.6 mm to (52.7, 66.0), turned to 270 degrees
- moved D8 28.3 mm to (45.7, 70.5), turned to 270 degrees
- moved R2 28.2 mm to (24.4, 60.6), turned to 90 degrees
- moved JP4 28.0 mm to (35.6, 81.3)
- moved Q1 17.9 mm to (27.9, 73.5)
- moved Q2 14.8 mm to (36.1, 64.9)
- moved JP7 13.2 mm to (18.2, 81.2)
- moved Q3 12.2 mm to (36.4, 55.2)
- moved Q4 11.6 mm to (30.9, 47.0)
- moved R1 11.5 mm to (17.8, 68.8), turned to 270 degrees
- moved D1 10.2 mm to (57.8, 14.0)
- moved R3 8.47 mm to (24.1, 29.2)
- moved JP8 7.85 mm to (31.6, 81.2)
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Connections:
- removed net N$1: LED1.K, R7.2
- removed net N$10: LED4.K, R6.2
- removed net N$16: LED5.K, R9.2
- removed net N$8: LED2.K, R8.1
- removed net N$9: LED3.K, R5.1
- removed net V3.3: JP1.6, JP10.1, JP11.1, JP4.1, JP5.1
- net 12V: no longer LED5.A
- net A+: no longer LED1.A, R8.2
- net A-: no longer LED2.A, R7.1
- net B+: no longer LED4.A, R5.2
- net B-: no longer LED3.A, R6.1
- net GND: now also JP3.1; no longer R9.1
- net N$13: now also JP3.3; no longer JP1.3, JP9.1
- net N$14: now also JP3.2; no longer JP1.2, JP12.1
- net N$15: now also JP4.1
- net N$6: now also JP3.5; no longer JP1.5, JP3.1
- net N$7: now also JP3.4; no longer JP1.4, JP6.1
Routing:
- net V3.3: track 72.4 -> 0.00 mm
- net 12V: track 125.0 -> 169.3 mm, vias 3 -> 0
- net A-: track 106.1 -> 64.0 mm, vias 2 -> 0
- net B-: track 113.3 -> 76.2 mm
- net N$6: track 92.1 -> 65.7 mm, vias 0 -> 2
- net B+: track 72.2 -> 54.3 mm
- net N$9: track 14.2 -> 0.00 mm
- net N$13: track 88.5 -> 76.9 mm, vias 1 -> 2
- net A+: track 97.0 -> 86.0 mm
- net N$7: track 70.0 -> 60.8 mm, vias 2 -> 0
- net N$1: track 7.41 -> 0.00 mm
- net N$15: track 10.9 -> 17.4 mm
- net N$8: track 5.50 -> 0.00 mm
- net N$16: track 5.50 -> 0.00 mm
- net N$10: track 5.24 -> 0.00 mm
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Other:
- board size 76.2 x 76.8 mm -> 76.2 x 90.2 mm
- board text added: "0603 PKG"
- board text added: "1N4001GP-E3"
- board text added: "20 VDC MAXIMUM ON GATES"
- board text added: "Dual H-Bridge August 2017 Lafe Spietz PUBLIC DOMAIN NO COPYRIGHT NO PATENTS"
- board text added: "IRF7862TRPBF"
- board text added: "ON/OFF SWITCH"
- board text added: "POWER IN (30VDC MAX)"
- board text added: "Vin"
- board text removed: "-"
- board text removed: "3.3V"
- board text removed: "3.3k"
- board text removed: "BUTTON"
- board text removed: "IRF7862"
- board text removed: "LED"
- board text removed: "NO PATENTS NO COPYRIGHTS NO MONEY NO MINING NO PROPERTY"
- board text removed: "ON"
- board text removed: "ON/OFF"
- board text removed: "POWER"
- board text removed: "STEPPER MOTOR CONTROL"

Commit message: repeated attempts to make gerber files that work
Parts:
- added JP5, JP6: M01PTH, SparkFun-Connectors:1X01
- added LED1: (no value), SparkFun-LED:LED5MM
- added R5: 3.3k, SparkFun-Passives:0603-RES
Connections:
- new net N$4: LED1.K, R5.2
- net 12V: now also LED1.A
- net GND: now also JP5.1, R5.1
- net N$15: now also JP6.1
Routing:
- net N$15: track 17.4 -> 105.4 mm
- net 12V: track 169.3 -> 182.6 mm
- net N$4: track 0.00 -> 4.86 mm
Other:
- board text added: "3.3k"
- board text added: "LED"
- board text added: "ON"
- board text added: "PWR"
Changed lines of the file:
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@@
 <text x="-7.62" y="-5.08" size="2.286" layer="27">Arduino Wee v1.3</text>
 <text x="2.54" y="-2.54" size="1.778" layer="27">Tent Vias!</text>
-<text x="18.415" y="67.945" size="1.778" layer="21">10k</text>
+<text x="19.05" y="67.945" size="1.778" layer="21">10k</text>
 <text x="19.05" y="59.69" size="1.778" layer="21">10k</text>
 <text x="15.875" y="1.905" size="1.778" layer="21">10k</text>
 <text x="24.765" y="27.305" size="1.778" layer="21">10k</text>
-<text x="3.81" y="34.29" size="1.778" layer="21">GND</text>
+<text x="4.445" y="35.56" size="1.778" layer="21">GND</text>
 <text x="24.13" y="83.82" size="1.778" layer="21">POWER IN
 (30VDC MAX)</text>
@@
 <text x="24.765" y="76.835" size="1.778" layer="21" rot="R180">GND</text>
 <text x="51.435" y="57.785" size="1.778" layer="21">V+</text>
-<text x="27.94" y="50.165" size="1.778" layer="21" rot="R180">GND</text>
+<text x="27.305" y="50.165" size="1.778" layer="21" rot="R180">GND</text>
 <text x="27.305" y="62.23" size="1.778" layer="21">2</text>
 <text x="36.195" y="59.055" size="1.778" layer="21">V+</text>
@@
 <wire x1="60.96" y1="7.62" x2="67.31" y2="13.97" width="0.4064" layer="21"/>
 <wire x1="67.31" y1="13.97" x2="67.31" y2="27.305" width="0.4064" layer="21"/>
-<wire x1="27.305" y1="3.81" x2="20.32" y2="3.81" width="0.4064" layer="21"/>
-<wire x1="20.32" y1="3.81" x2="20.32" y2="22.225" width="0.4064" layer="21"/>
+<wire x1="27.305" y1="4.445" x2="20.32" y2="4.445" width="0.4064" layer="21"/>
+<wire x1="20.32" y1="4.445" x2="20.32" y2="22.225" width="0.4064" layer="21"/>
 <wire x1="20.32" y1="22.225" x2="20.32" y2="38.735" width="0.4064" layer="21"/>
 <wire x1="20.32" y1="38.735" x2="18.415" y2="38.735" width="0.4064" layer="21"/>
@@
 <text x="13.335" y="65.405" size="1.778" layer="21">0603 PKG</text>
 <text x="40.005" y="79.375" size="1.778" layer="22" rot="MR0">Vin</text>
-<text x="18.415" y="11.43" size="1.778" layer="21" rot="R90">Dual H-Bridge
+<text x="16.51" y="15.24" size="1.778" layer="21" rot="R90">Dual H-Bridge
 August 2017
 Lafe Spietz
@@
 <text x="55.245" y="2.54" size="1.778" layer="21" rot="R180">GND</text>
 <text x="30.48" y="40.005" size="1.778" layer="21" rot="R180">GND</text>
-<text x="29.21" y="9.525" size="1.778" layer="21" rot="R180">GND</text>
+<text x="28.575" y="9.525" size="1.778" layer="21" rot="R180">GND</text>
 <hole x="24.13" y="81.28" drill="3.2"/>
+<wire x1="65.405" y1="69.85" x2="65.405" y2="71.755" width="0.4064" layer="21"/>
+<wire x1="65.405" y1="71.755" x2="65.405" y2="73.025" width="0.4064" layer="21"/>
+<wire x1="65.405" y1="73.025" x2="65.405" y2="74.295" width="0.4064" layer="21"/>
+<wire x1="65.405" y1="74.295" x2="65.405" y2="75.565" width="0.4064" layer="21"/>
+<wire x1="65.405" y1="75.565" x2="65.405" y2="77.47" width="0.4064" layer="21"/>
+<wire x1="65.405" y1="77.47" x2="73.66" y2="77.47" width="0.4064" layer="21"/>
+<wire x1="73.66" y1="77.47" x2="73.66" y2="75.565" width="0.4064" layer="21"/>
+<wire x1="73.66" y1="75.565" x2="73.66" y2="74.295" width="0.4064" layer="21"/>
+<wire x1="73.66" y1="74.295" x2="73.66" y2="73.025" width="0.4064" layer="21"/>
+<wire x1="73.66" y1="73.025" x2="73.66" y2="71.755" width="0.4064" layer="21"/>
+<wire x1="73.66" y1="71.755" x2="73.66" y2="69.85" width="0.4064" layer="21"/>
+<wire x1="73.66" y1="69.85" x2="65.405" y2="69.85" width="0.4064" layer="21"/>
+<wire x1="66.675" y1="70.485" x2="67.31" y2="70.485" width="0.4064" layer="21"/>
+<wire x1="67.31" y1="70.485" x2="67.945" y2="70.485" width="0.4064" layer="21"/>
+<wire x1="66.675" y1="76.835" x2="67.31" y2="76.835" width="0.4064" layer="21"/>
+<wire x1="67.31" y1="76.835" x2="67.945" y2="76.835" width="0.4064" layer="21"/>
+<wire x1="67.31" y1="76.835" x2="67.31" y2="74.295" width="0.4064" layer="21"/>
+<wire x1="67.31" y1="74.295" x2="67.31" y2="73.025" width="0.4064" layer="21"/>
+<wire x1="67.31" y1="73.025" x2="67.31" y2="70.485" width="0.4064" layer="21"/>
+<wire x1="72.39" y1="76.835" x2="71.755" y2="76.835" width="0.4064" layer="21"/>
+<wire x1="71.755" y1="76.835" x2="71.12" y2="76.835" width="0.4064" layer="21"/>
+<wire x1="71.755" y1="76.835" x2="71.755" y2="74.295" width="0.4064" layer="21"/>
+<wire x1="71.755" y1="74.295" x2="71.755" y2="73.025" width="0.4064" layer="21"/>
+<wire x1="71.755" y1="73.025" x2="71.755" y2="70.485" width="0.4064" layer="21"/>
+<wire x1="71.12" y1="70.485" x2="72.39" y2="70.485" width="0.4064" layer="21"/>
+<wire x1="67.31" y1="74.295" x2="71.755" y2="74.295" width="0.4064" layer="21"/>
+<wire x1="71.755" y1="73.025" x2="67.31" y2="73.025" width="0.4064" layer="21"/>
+<wire x1="65.405" y1="75.565" x2="66.675" y2="75.565" width="0.4064" layer="21"/>
+<wire x1="65.405" y1="74.295" x2="66.675" y2="74.295" width="0.4064" layer="21"/>
+<wire x1="65.405" y1="73.025" x2="66.675" y2="73.025" width="0.4064" layer="21"/>
+<wire x1="65.405" y1="71.755" x2="66.675" y2="71.755" width="0.4064" layer="21"/>
+<wire x1="72.39" y1="75.565" x2="73.66" y2="75.565" width="0.4064" layer="21"/>
+<wire x1="72.39" y1="74.295" x2="73.66" y2="74.295" width="0.4064" layer="21"/>
+<wire x1="72.39" y1="73.025" x2="73.66" y2="73.025" width="0.4064" layer="21"/>
+<wire x1="72.39" y1="71.755" x2="73.66" y2="71.755" width="0.4064" layer="21"/>
+<hole x="15.24" y="6.985" drill="3.2"/>
+<text x="17.78" y="11.43" size="1.778" layer="21" rot="R270">GND</text>
+<text x="10.16" y="11.43" size="1.778" layer="21" rot="R270">PWR</text>
+<text x="71.755" y="54.61" size="1.778" layer="21">ON</text>
+<text x="67.31" y="55.245" size="1.778" layer="21" rot="R270">3.3k</text>
+<text x="67.945" y="62.865" size="1.778" layer="21">LED</text>
 </plain>
 <attributes>
@@
 <element name="JP1" library="SparkFun-Connectors" package="1X01" value="M01PTH" x="15.24" y="81.28"/>
 <element name="JP4" library="SparkFun-Connectors" package="1X01" value="M01PTH" x="35.56" y="81.28"/>
+<element name="JP5" library="SparkFun-Connectors" package="1X01" value="M01PTH" x="17.78" y="12.7"/>
+<element name="JP6" library="SparkFun-Connectors" package="1X01" value="M01PTH" x="12.065" y="12.7"/>
+<element name="LED1" library="SparkFun-LED" package="LED5MM" value="" x="70.485" y="59.055" rot="R270"/>
+<element name="R5" library="SparkFun-Passives" package="0603-RES" value="3.3k" x="70.485" y="52.07" rot="R90"/>
 </elements>
 <signals>
@@
 <polygon width="0.254" layer="16" isolate="0.3048">
 <vertex x="0" y="91.44"/>
-<vertex x="76.2" y="91.44"/>
+<vertex x="76.2" y="90.805"/>
 <vertex x="76.2" y="0"/>
 <vertex x="0" y="0"/>
@@
 <contactref element="JP3" pad="1"/>
 <contactref element="JP1" pad="1"/>
+<contactref element="JP5" pad="1"/>
+<contactref element="R5" pad="1"/>
 </signal>
 <signal name="N$30">
@@
 <wire x1="39.1922" y1="59.69" x2="52.705" y2="59.69" width="0.8128" layer="1"/>
 <wire x1="52.705" y1="59.69" x2="52.705" y2="60.96" width="0.8128" layer="1"/>
+<contactref element="LED1" pad="A"/>
+<wire x1="70.485" y1="60.325" x2="57.15" y2="60.325" width="0.8128" layer="16"/>
 </signal>
 <signal name="A-">
@@
 <wire x1="32.385" y1="80.645" x2="32.385" y2="81.153" width="0.4064" layer="1"/>
 <wire x1="32.385" y1="81.153" x2="31.623" y2="81.153" width="0.4064" layer="1"/>
+<contactref element="JP6" pad="1"/>
+<wire x1="12.065" y1="12.7" x2="12.065" y2="37.465" width="0.8128" layer="16"/>
+<wire x1="12.065" y1="37.465" x2="31.623" y2="37.465" width="0.8128" layer="16"/>
+<wire x1="31.623" y1="37.465" x2="31.623" y2="81.153" width="0.8128" layer="16"/>
 </signal>
 <signal name="N$1">
 </signal>
+<signal name="N$4">
+<contactref element="LED1" pad="K"/>
+<contactref element="R5" pad="2"/>
+<wire x1="70.485" y1="52.92" x2="70.485" y2="57.785" width="0.8128" layer="1"/>
+</signal>
 </signals>
